Commit message: Added ultrasound to the urdf and updated the sonar topic name in the yaml file.

File: bv80bot/neato_robot/neato_node/urdf/neato.urdf.xacro (robot description, xacro)
@@ -23,3 +23,29 @@
        <child link="base_link" />
    </joint>
+    <joint name="ultrasound_top_joint" type="fixed">
+      <parent link="base_link"/>
+      <child link="ultrasound_top"/>
+      <origin xyz="0.051 0 0.343" rpy="0 0 0"/>
+    </joint>
+    <link name="ultrasound_top">
+      <!--visual>
+        <geometry>
+          <mesh filename="package://kobuki_description/meshes/wheel.dae"/>
+        </geometry>
+        <origin xyz="0 0 0" rpy="0 0 0"/>
+      </visual-->
+      <!--collision>
+        <geometry>
+          <cylinder length="0.0206" radius="0.0352"/>
+        </geometry>
+        <origin rpy="0 0 0" xyz="0 0 0"/>
+      </collision-->
+      <inertial>
+        <mass value="0.01" />
+        <origin xyz="0 0 0" />
+        <inertia ixx="0.001" ixy="0.0" ixz="0.0"
+                 iyy="0.001" iyz="0.0"
+                 izz="0.001" />
+      </inertial>
+    </link>
 </robot>
